Commit message: Working on bicycle controlled robots in sim

File: src/hunter_sim/hunter2_gazebo/xacro/lidar.xacro (robot description, xacro)
@@ -29,5 +29,5 @@
     </link>
 <gazebo reference="laser_frame">
-    <material>Gazebo/Red</material>
+    <material>Gazebo/Grey</material>
     <sensor name="laser" type="gpu_ray">
     <pose> 0 0 0 0 0 0 </pose>
