Commit message: Working version for day2 with lelr at CSA

File: src/hunter_sim/hunter2_gazebo/xacro/hunter2_gazebo_lidar.xacro (robot description, xacro)
@@ -6,8 +6,8 @@
   <joint name="laser_joint" type="fixed">
     <parent link="base_link" />
-    <child link="laser_frame" />
+    <child link="lidar_link" />
     <origin xyz="0.05 0 0.05" rpy="0 0 0" />
   </joint>
-  <link name="laser_frame">
+  <link name="lidar_link">
     <inertial>
       <origin xyz="0 0 0" rpy="0 0 0" />
@@ -31,5 +31,5 @@
     </collision>
   </link>
-  <gazebo reference="laser_frame">
+  <gazebo reference="lidar_link">
     <material>Gazebo/Grey</material>
     <sensor name="laser" type="gpu_ray">
@@ -38,5 +38,5 @@
       <update_rate>10</update_rate>
       <topic>$(arg namespace)/scan</topic>
-      <gz_frame_id>$(arg namespace)/laser_frame</gz_frame_id>
+      <gz_frame_id>$(arg namespace)/lidar_link</gz_frame_id>
       <lidar>
         <scan>
