Commit message: Update mass and namespaces

File: src/hunter_sim/hunter2_base/urdf/hunter2_base.xacro (robot description, xacro)
@@ -4,4 +4,21 @@
   <!-- Base Link -->
   <link name="base_link">
+    <visual>
+      <origin xyz="0 0 0" rpy="0 0 0" />
+      <geometry>
+        <mesh filename="package://hunter2_base/meshes/base_link.STL" />
+      </geometry>
+      <material name="body">
+        <color rgba="$(arg body_colour)" />
+      </material>
+    </visual>
+    <collision>
+      <origin xyz="0 0 0" rpy="0 0 0" />
+      <geometry>
+        <mesh filename="package://hunter2_base/meshes/base_link.STL" />
+      </geometry>
+    </collision>
+  </link>
+  <link name="base_link2">
     <inertial>
       <origin xyz="0.0266989327622036 0.000409203500587652 -0.135901124750884" rpy="0 0 0" />
@@ -11,20 +28,9 @@
         iyy="0.111072002332437" iyz="-5.13308150598312E-07" izz="0.12660862809283" />
     </inertial>
-    <visual>
-      <origin xyz="0 0 0" rpy="0 0 0" />
-      <geometry>
-        <mesh filename="package://hunter2_base/meshes/base_link.STL" />
-      </geometry>
-      <material name="body">
-        <color rgba="$(arg body_colour)" />
-      </material>
-    </visual>
-    <collision>
-      <origin xyz="0 0 0" rpy="0 0 0" />
-      <geometry>
-        <mesh filename="package://hunter2_base/meshes/base_link.STL" />
-      </geometry>
-    </collision>
-  </link>
+  </link>
+  <joint name="dummy_base" type="fixed">
+    <parent link="base_link" />
+    <child link="base_link2" />
+  </joint>
   <!-- Front Left Steering Link & Joint -->
   <link name="front_steer_left_link">
